File: Hardware/nard_sam.kicad_pcb (KiCad board)
At the start: 4 copper layers, 63.5 x 21 mm, 29 parts, among them J1 SIM_Card, J2 SIM_Card, J3 Conn_01x08, J4 Conn_01x10, J5 Conn_01x04, J6 M20-7910842R, J7 M20-7911042R, U1 SEC1210, U3 ST4SIM-200M

Commit message: switched from 4-to-2 layer PCB
Routing:
- net +5V: track 37.4 -> 93.2 mm, vias 3 -> 2
- removed copper zone on In2.Cu, net +5V
- removed copper zone on In1.Cu, net GND
Other:
- copper layers 4 -> 2
Changed lines of the file:
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@@
 	(layers
 		(0 "F.Cu" signal)
-		(1 "In1.Cu" signal)
-		(2 "In2.Cu" signal)
 		(31 "B.Cu" signal)
 		(32 "B.Adhes" user "B.Adhesive")
@@
 			(layer "dielectric 1"
 				(type "core")
-				(thickness 0.2)
-				(material "FR4")
-				(epsilon_r 4.5)
-				(loss_tangent 0.02)
-			)
-			(layer "In1.Cu"
-				(type "copper")
-				(thickness 0.00175)
-			)
-			(layer "dielectric 2"
-				(type "prepreg")
-				(thickness 1.065)
-				(material "FR4")
-				(epsilon_r 4.5)
-				(loss_tangent 0.02)
-			)
-			(layer "In2.Cu"
-				(type "copper")
-				(thickness 0.00175)
-			)
-			(layer "dielectric 3"
-				(type "core")
-				(thickness 0.2)
+				(thickness 1.4685)
 				(material "FR4")
 				(epsilon_r 4.5)
@@
 	)
 	(via
-		(at 74.11 74.3276)
-		(size 0.8)
-		(drill 0.4)
-		(layers "F.Cu" "B.Cu")
-		(net 5)
-	)
-	(via
 		(at 110.675 72.55)
 		(size 0.8)
@@
 	)
 	(segment
+		(start 108.375 72.474695)
+		(end 108.839 72.010695)
+		(width 0.25)
+		(layer "B.Cu")
+		(net 5)
+	)
+	(segment
 		(start 74.11 74.3276)
 		(end 74.11 70.345)
@@
 	)
 	(segment
+		(start 108.839 69.839305)
+		(end 107.3078 68.308105)
+		(width 0.25)
+		(layer "B.Cu")
+		(net 5)
+	)
+	(segment
+		(start 104.9528 62.7634)
+		(end 104.9528 61.1378)
+		(width 0.25)
+		(layer "B.Cu")
+		(net 5)
+	)
+	(segment
+		(start 108.839 72.010695)
+		(end 108.839 69.839305)
+		(width 0.25)
+		(layer "B.Cu")
+		(net 5)
+	)
+	(segment
+		(start 107.575 65.5188)
+		(end 107.575 63.474695)
+		(width 0.25)
+		(layer "B.Cu")
+		(net 5)
+	)
+	(segment
+		(start 108.375 73.075305)
+		(end 108.375 72.474695)
+		(width 0.25)
+		(layer "B.Cu")
+		(net 5)
+	)
+	(segment
 		(start 97.8 78.7)
 		(end 78.5 78.7)
@@
 	)
 	(segment
+		(start 106.863705 62.7634)
+		(end 104.9528 62.7634)
+		(width 0.25)
+		(layer "B.Cu")
+		(net 5)
+	)
+	(segment
+		(start 75.692 60.833)
+		(end 73.025 63.5)
+		(width 0.25)
+		(layer "B.Cu")
+		(net 5)
+	)
+	(segment
+		(start 73.025 66.695)
+		(end 74.11 67.78)
+		(width 0.25)
+		(layer "B.Cu")
+		(net 5)
+	)
+	(segment
 		(start 78.5 78.7)
 		(end 74.1276 74.3276)
@@
 	)
 	(segment
+		(start 104.648 60.833)
+		(end 75.692 60.833)
+		(width 0.25)
+		(layer "B.Cu")
+		(net 5)
+	)
+	(segment
 		(start 74.1276 74.3276)
 		(end 74.11 74.3276)
@@
 	)
 	(segment
+		(start 73.025 63.5)
+		(end 73.025 66.695)
+		(width 0.25)
+		(layer "B.Cu")
+		(net 5)
+	)
+	(segment
+		(start 109.725 73.5)
+		(end 108.799695 73.5)
+		(width 0.25)
+		(layer "B.Cu")
+		(net 5)
+	)
+	(segment
+		(start 107.3078 68.308105)
+		(end 107.3078 65.786)
+		(width 0.25)
+		(layer "B.Cu")
+		(net 5)
+	)
+	(segment
+		(start 107.575 63.474695)
+		(end 106.863705 62.7634)
+		(width 0.25)
+		(layer "B.Cu")
+		(net 5)
+	)
+	(segment
+		(start 104.9528 61.1378)
+		(end 104.648 60.833)
+		(width 0.25)
+		(layer "B.Cu")
+		(net 5)
+	)
+	(segment
 		(start 74.11 70.345)
 		(end 74.11 67.78)
@@
 	)
 	(segment
+		(start 108.799695 73.5)
+		(end 108.375 73.075305)
+		(width 0.25)
+		(layer "B.Cu")
+		(net 5)
+	)
+	(segment
+		(start 107.3078 65.786)
+		(end 107.575 65.5188)
+		(width 0.25)
+		(layer "B.Cu")
+		(net 5)
+	)
+	(segment
+		(start 110.675 72.55)
+		(end 109.725 73.5)
+		(width 0.25)
+		(layer "B.Cu")
+		(net 5)
+	)
+	(segment
 		(start 76.65 73.655)
 		(end 76.65 67.78)
@@
 	(segment
 		(start 104.4194 66.3166)
-		(end 105.0544 66.3166)
-		(width 0.25)
-		(layer "F.Cu")
-		(net 34)
-	)
-	(segment
-		(start 105.0544 66.3166)
 		(end 105.3084 66.3166)
 		(width 0.25)
@@
 	(segment
 		(start 104.099 66.637)
-		(end 104.267 66.469)
+		(end 104.4194 66.3166)
 		(width 0.25)
 		(layer "F.Cu")
@@
 		(net 34)
 	)
-	(segment
-		(start 104.267 66.469)
-		(end 104.4194 66.3166)
-		(width 0.25)
-		(layer "F.Cu")
-		(net 34)
-	)
 	(via
 		(at 105.9942 65.6308)
@@
 	)
 	(segment
-		(start 106.557495 71.2326)
+		(start 105.9942 70.669305)
 		(end 107.0102 71.685305)
 		(width 0.25)
@@
 	)
 	(segment
-		(start 105.9942 70.669305)
-		(end 106.557495 71.2326)
-		(width 0.25)
-		(layer "B.Cu")
-		(net 34)
-	)
-	(segment
 		(start 105.9942 65.6308)
 		(end 105.9942 70.669305)
@@
 	)
 	(segment
-		(start 102.149 67.324)
-		(end 102.125 67.3)
-		(width 0.25)
-		(layer "F.Cu")
-		(net 38)
-	)
-	(segment
-		(start 102.149 67.4845)
-		(end 102.149 67.324)
-		(width 0.25)
-		(layer "F.Cu")
-		(net 38)
-	)
-	(segment
 		(start 91.928 73.613)
 		(end 96.337 73.613)
@@
 		(hatch edge 0.508)
 		(connect_pads
-			(clearance 0.508)
-		)
-		(min_thickness 0.254)
-		(filled_areas_thickness no)
-		(fill yes
-			(thermal_gap 0.508)
-			(thermal_bridge_width 0.508)
-		)
-		(polygon
-			(pts
-				(xy 136.25 82.5) (xy 70.25 82.5) (xy 70.25 56.5) (xy 136.25 56.5)
-			)
-		)
-	)
-	(zone
-		(net 12)
-		(net_name "GND")
-		(layer "In1.Cu")
-		(hatch edge 0.508)
-		(connect_pads
-			(clearance 0.508)
-		)
-		(min_thickness 0.254)
-		(filled_areas_thickness no)
-		(fill yes
-			(thermal_gap 0.508)
-			(thermal_bridge_width 0.508)
-		)
-		(polygon
-			(pts
-				(xy 136.25 82.5) (xy 70.25 82.5) (xy 70.25 56.5) (xy 136.25 56.5)
-			)
-		)
-	)
-	(zone
-		(net 5)
-		(net_name "+5V")
-		(layer "In2.Cu")
-		(hatch edge 0.508)
-		(connect_pads
